File: breakout_board/breakout_board.sch (KiCad schematic (older format))
At the start: 54 parts, among them J1 Conn_01x14, J2 Conn_01x14, J3 CONN_01X03, J4 CONN_02x04, J5 Conn_01x04, U1 TB6612FNG, U2 LP5907SNX-3.3/NOPB, U3 LSF0204RUTR, U4 ADP3330, U5 TLV70718PDQNR

Commit message: Fixed board
Parts:
- MICRO1: footprint footprints:ATMEGA32U4-MUR -> Housings_DFN_QFN:QFN-44-1EP_7x7mm_Pitch0.5mm
Connections:
- net +5V: now also U3.12 (EN)
- no-connect marks 9 -> 11
Other:
- note added: "EN was not connected to Vref_B"
Changed lines of the file:
@@
 F 0 "MICRO1" H 2750 7350 50  0000 C CNN
 F 1 "ATMEGA32U4-MU" H 4400 4150 50  0000 C CNN
-F 2 "footprints:ATMEGA32U4-MUR" H 3700 5650 50  0001 C CIN
+F 2 "Housings_DFN_QFN:QFN-44-1EP_7x7mm_Pitch0.5mm" H 3700 5650 50  0001 C CIN
 F 3 "" H 4800 6750 50  0001 C CNN
 	1    3700 5650
@@
 	9700 5400 9700 5600
 NoConn ~ 9700 5800
+Connection ~ 10150 3050
+NoConn ~ 1300 3900
+NoConn ~ 1800 4100
+Text Notes 10225 3050 0    60   ~ 0
+EN was not connected to Vref_B
 $EndSCHEMATC

Commit message: made kicad v2
ditched altium due to poor generic component libraries (depends heavily
on vault), doing a 2-layer layout.
Parts:
- J4: symbol Conn_02x04_Counter_Clockwise -> Conn_02x04_Counter_Clockwise-RESCUE-breakout_board
- MICRO1: footprint Housings_DFN_QFN:QFN-44-1EP_7x7mm_Pitch0.5mm -> footprints:QFN-44-1EP_7x7mm_Pitch0.5mm_M
Connections:
- net +3V3: now also J4.7 (Pin_4); no longer J4.4 (Pin_4)
- net GND: now also J4.8 (Pin_5); no longer J4.5 (Pin_5)
- net IO8: now also J4.5 (Pin_3); no longer J4.3 (Pin_3)
- net MISO: now also J4.2 (Pin_8); no longer J4.8 (Pin_8)
- net MOSI: now also J4.3 (Pin_2); no longer J4.2 (Pin_2)
- net SCK: now also J4.4 (Pin_7); no longer J4.7 (Pin_7)
Changed lines of the file:
@@
 EESchema Schematic File Version 2
+LIBS:breakout_board-rescue
 LIBS:power
 LIBS:device
@@
 F 0 "MICRO1" H 2750 7350 50  0000 C CNN
 F 1 "ATMEGA32U4-MU" H 4400 4150 50  0000 C CNN
-F 2 "Housings_DFN_QFN:QFN-44-1EP_7x7mm_Pitch0.5mm" H 3700 5650 50  0001 C CIN
+F 2 "footprints:QFN-44-1EP_7x7mm_Pitch0.5mm_M" H 3700 5650 50  0001 C CIN
 F 3 "" H 4800 6750 50  0001 C CNN
 	1    3700 5650
@@
 BLDC HEADER
 $Comp
-L Conn_02x04_Counter_Clockwise J4
+L Conn_02x04_Counter_Clockwise-RESCUE-breakout_board J4
 U 1 1 59D1D857
 P 4200 1200
@@
 NoConn ~ 1300 3900
 NoConn ~ 1800 4100
-Text Notes 10225 3050 0    60   ~ 0
+Text Notes 9625 2550 0    60   ~ 0
 EN was not connected to Vref_B
 $EndSCHEMATC
