File: breakout_board/_saved_breakout_board.sch (KiCad schematic (older format))
At the start: 54 parts, among them J1 Conn_01x14, J2 Conn_01x14, J3 CONN_01X03, J4 CONN_02x04, J5 Conn_01x04, U1 TB6612FNG, U2 LP5907SNX-3.3/NOPB, U3 LSF0204RUTR, U4 ADP3330, U5 TLV70718PDQNR

Commit message: Changed components, routed a bunch of stuff
Connections:
- net SCL is gone; now on net D3/SCL: MICRO1.18 ((OC0B/SCL/INT0)PD0)
- net SDA is gone; now on net D2/SDA: MICRO1.19 ((SDA/INT1)PD1)
Changed lines of the file:
@@
 D5*
 Text Label 4800 5300 0    60   ~ 0
-SCL
+D3/SCL
 Text Label 4800 5400 0    60   ~ 0
-SDA
+D2/SDA
 Text Label 4800 5500 0    60   ~ 0
 D0/RX
