File: breakout_board/_saved_breakout_board.sch (KiCad schematic (older format))
At the start: 54 parts, among them J1 Conn_01x14, J2 Conn_01x14, J3 CONN_01X03, J4 CONN_02x04, J5 Conn_01x04, U1 TB6612FNG, U2 LP5907SNX-3.3/NOPB, U3 LSF0204RUTR, U4 ADP3330, U5 TLV70718PDQNR

Commit message: Fixed board
Parts:
- MICRO1: footprint Housings_DFN_QFN:QFN-44-1EP_7x7mm_Pitch0.5mm -> footprints:QFN-44-1EP_7x7mm_Pitch0.5mm_M
Changed lines of the file:
@@
 F 0 "MICRO1" H 2750 7350 50  0000 C CNN
 F 1 "ATMEGA32U4-MU" H 4400 4150 50  0000 C CNN
-F 2 "Housings_DFN_QFN:QFN-44-1EP_7x7mm_Pitch0.5mm" H 3700 5650 50  0001 C CIN
+F 2 "footprints:QFN-44-1EP_7x7mm_Pitch0.5mm_M" H 3700 5650 50  0001 C CIN
 F 3 "" H 4800 6750 50  0001 C CNN
 	1    3700 5650
