File: breakout_board/breakout_board.kicad_pcb (KiCad board)
At the start: 2 copper layers, 52 parts, among them J1 CONN_01X17, J2 CONN_01X17, J3 CONN_01X03, J4 CONN_02x04, U1 TB6612FNG, U2 LP5907SNX-3.3/NOPB, U3 LSF0204RUTR

Commit message: More done
Parts:
- added J5: Conn_01x04, Pin_Headers:Pin_Header_Straight_1x04_Pitch2.54mm, F.Cu at (197.5, 25.2)
- J1, J2: value CONN_01X17 -> Conn_01x14
- J4: footprint Pin_Headers:Pin_Header_Straight_2x03_Pitch2.54mm_SMD -> Pin_Headers:Pin_Header_Straight_2x04_Pitch2.54mm_SMD
- moved U3 151.9 mm to (40.5, 55.2)
- moved LED3 125.8 mm to (41.2, 82.2)
- moved J1 123.4 mm to (217.5, 31.2)
- moved D1 114.8 mm to (195.2, 54.0), turned to 90 degrees
- moved IND1 111.2 mm to (189.5, 53.0), turned to 90 degrees
- moved OS1 109.3 mm to (200.8, 50.0), turned to 180 degrees
- moved C1 106.8 mm to (203.2, 50.2), turned to 270 degrees
- moved R7 101.7 mm to (98.2, 32.2)
- moved U1 101.1 mm to (194.2, 37.2), turned to 270 degrees
- moved C10 100.4 mm to (82.0, 39.2)
- moved R2 100.3 mm to (52.8, 98.5)
- moved C2 99.8 mm to (198.5, 51.5), turned to 270 degrees
- moved LED1 95.9 mm to (55.5, 85.5)
- moved LED2 94.6 mm to (115.5, 66.0)
- moved C18 94.3 mm to (68.8, 96.5)
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Connections:
- BTN1 pad 1: GND -> Net-(BTN1-Pad1)
- BTN1 pad 2: Net-(BTN1-Pad2) -> /RESET
- BTN1 pad 3: Net-(BTN1-Pad3) -> GND
- BTN1 pad 4: /RESET -> Net-(BTN1-Pad4)
- J1 pad 1: /MOSI -> /RESET
- J1 pad 10: Net-(J1-Pad10) -> /D3/SCL
- J1 pad 11: Net-(J1-Pad11) -> /D2/SDA
- J1 pad 12: /D7 -> /IO11*
- J1 pad 13: /IO8 -> /MISO
- J1 pad 14: /IO9* -> /MOSI
- J1 pad 2: /RXLED/SS -> /IO10*
- J1 pad 3: /D1/TX -> /IO9*
- J1 pad 4: /D0/RX -> /IO8
- J1 pad 5: /RESET -> /IO12*
- J1 pad 6: GND -> /D1/TX
- J1 pad 7: /D2/SDA -> /D0/RX
- J1 pad 8: /D3/SCL -> GND
- J1 pad 9: Net-(J1-Pad9) -> /RESET
- J2 pad 1: /SCK -> /IO13*
- J2 pad 10: /A4 -> GND
- J2 pad 11: /A3 -> /D7
- J2 pad 12: /A2 -> +12V
- J2 pad 13: /A1 -> /RXLED/SS
- J2 pad 14: /A0 -> /SCK
- J2 pad 2: /MISO -> +5V
- J2 pad 3: +12V -> /A0
- J2 pad 4: GND -> /A1
- J2 pad 5: /RESET -> /A2
- J2 pad 6: +5V -> /A3
- J2 pad 7: Net-(J2-Pad7) -> /A4
- J2 pad 8: Net-(J2-Pad8) -> /A5
- J2 pad 9: /A5 -> /AREF
- J4 pad 2: /MOSI -> /MISO
- J4 pad 3: /IO8 -> /MOSI
- J4 pad 4: +3V3 -> /SCK
- J4 pad 5: GND -> /IO8
- V_REG_1V8 pad 2: +1V8 -> (no net)

Commit message: worked some more
Parts:
- moved U3 162.2 mm to (202.4, 46.0), turned to 90 degrees
- moved C16 146.0 mm to (199.6, 41.9), turned to 90 degrees
- moved C15 130.4 mm to (186.9, 41.7), turned to 270 degrees
- moved R9 119.9 mm to (206.8, 47.2), turned to 270 degrees
- moved C13 114.5 mm to (189.7, 57.1), turned to 90 degrees
- moved C14 112.9 mm to (188.5, 41.7), turned to 270 degrees
- moved R7 100.6 mm to (195.6, 57.7)
- moved R8 95.3 mm to (205.0, 47.2), turned to 270 degrees
- moved J4 91.6 mm to (189.7, 64.5), turned to 180 degrees
- moved C17 90.4 mm to (201.7, 41.9), turned to 90 degrees
- moved R10 70.0 mm to (205.0, 44.5), turned to 90 degrees
- moved LSM6DS3US1 68.2 mm to (192.5, 56.4), turned to 270 degrees
- moved R11 61.1 mm to (200.2, 45.2), turned to 90 degrees
- moved R13 60.5 mm to (203.5, 41.9), turned to 90 degrees
- moved R12 59.8 mm to (200.2, 47.5), turned to 270 degrees
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
Commit message: Changed components, routed a bunch of stuff
Parts:
- removed V_REG1: NCP1117-5, footprints:NCP1117
- removed V_REG_1V8: NCP1117DT18RKG, footprints:TO229P990X238-4N
- added C20: 1uF, Capacitors_SMD:C_0603, F.Cu at (128.6, 103.6)
- added U4: ADP3330, TO_SOT_Packages_SMD:SOT-23-6, F.Cu at (136.3, 117.3)
- added U5: TLV70718PDQNR, footprints:DQN4, F.Cu at (130.1, 103.6)
- C7, C9: value 10uF -> 1uF; footprint Capacitors_SMD:C_0805 -> Capacitors_SMD:C_0603
- J4: moved to B.Cu
- moved LED3 110.5 mm to (146.6, 115.6), turned to 180 degrees
- moved LED1 94.8 mm to (146.6, 111.9), turned to 180 degrees
- moved C10 92.3 mm to (129.5, 118.4)
- moved R2 91.5 mm to (143.3, 112.0), turned to 180 degrees
- moved LED4 89.9 mm to (146.6, 117.3), turned to 180 degrees
- moved J1 84.9 mm to (151.4, 84.6)
- moved J5 80.1 mm to (143.0, 84.6)
- moved IND1 79.6 mm to (133.1, 109.2)
- moved C13 79.3 mm to (133.1, 112.6)
- moved R7 79.1 mm to (140.0, 113.9)
- moved LSM6DS3US1 78.9 mm to (136.1, 111.6)
- moved C8 78.8 mm to (135.4, 108.3)
- moved R1 78.7 mm to (141.2, 108.7)
- moved C6 78.1 mm to (139.8, 110.5)
- moved D1 78.0 mm to (139.7, 108.7)
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Connections:
- MICRO1 pad 18: /SCL -> /D3/SCL
- MICRO1 pad 19: /SDA -> /D2/SDA
Routing:
- net /MOSI: track 0.00 -> 56.1 mm, vias 0 -> 3
- net +5V: track 0.00 -> 41.4 mm, vias 0 -> 4
- net GND: track 0.00 -> 37.6 mm, vias 0 -> 7
- net /TXLED: track 0.00 -> 34.9 mm, vias 0 -> 2
- net /D5*: track 0.00 -> 26.7 mm, vias 0 -> 3
- net /HWB: track 0.00 -> 25.6 mm, vias 0 -> 2
- net /IO10*: track 0.00 -> 25.5 mm, vias 0 -> 2
- net /RESET: track 0.00 -> 22.0 mm, vias 0 -> 2
- net /IO9*: track 0.00 -> 20.5 mm, vias 0 -> 2
- net /MISO: track 0.00 -> 18.8 mm, vias 0 -> 1
- net /IO12*: track 0.00 -> 17.7 mm, vias 0 -> 2
- net /IO11*: track 0.00 -> 16.7 mm, vias 0 -> 1
- net /IO8: track 0.00 -> 16.3 mm
- net /A0: track 0.00 -> 15.9 mm
- net /D7: track 0.00 -> 13.7 mm, vias 0 -> 1
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- added copper zone on F.Cu, net +5V
- added copper zone on B.Cu, net GND
Other:
- board outline added: 30.2 x 37.9 mm
- copper layers 2 -> 4
- net class Custom added: clearance 0.1, trace_width 0.1524, via_dia 0.6, via_drill 0.4
- rule trace_min: 0.2 -> 0.15

Commit message: Finished the board layout
Parts:
- moved IMU 0.20 mm to (136.3, 111.8)
- turned R7 to 180 degrees
- turned C12 to 90 degrees
- renumbered LSM6DS3US1 to IMU
Routing:
- net GND: track 37.6 -> 161.1 mm, vias 7 -> 21
- net +5V: track 41.4 -> 110.2 mm, vias 4 -> 13
- net /SDA_1V8: track 0.00 -> 62.6 mm, vias 0 -> 4
- net +12V: track 2.89 -> 61.0 mm, vias 0 -> 5
- net /IO13*: track 0.00 -> 56.5 mm, vias 0 -> 3
- net /INT2: track 0.00 -> 51.7 mm, vias 0 -> 4
- net /RESET: track 22.0 -> 73.0 mm, vias 2 -> 3
- net +1V8: track 0.00 -> 44.0 mm, vias 0 -> 6
- net /IO8: track 16.3 -> 56.9 mm, vias 0 -> 4
- net /SCL_1V8: track 0.00 -> 40.0 mm, vias 0 -> 7
- net /SCK: track 8.41 -> 47.3 mm
- net /MISO: track 18.8 -> 54.4 mm, vias 1 -> 2
- net /INT1: track 0.00 -> 22.6 mm, vias 0 -> 4
- net /IO11*: track 16.7 -> 38.3 mm, vias 1 -> 2
- net /RXLED/SS: track 10.3 -> 27.4 mm
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- added copper zone on In2.Cu, net +1V8
- added copper zone on In1.Cu, net +3V3
Other:
- board text added: "+12V"
- board text added: "+5V"
- board text added: "A0"
- board text added: "A1"
- board text added: "A2"
- board text added: "A3"
- board text added: "A4"
- board text added: "A5"
- board text added: "AREF"
- board text added: "D7"
- board text added: "GND"
- board text added: "IO10*"
- board text added: "IO11*"
- board text added: "IO12*"
- board text added: "IO13*"
- board text added: "IO8"
- board text added: "IO9*"
- board text added: "MISO"
- board text added: "MOSI"
- board text added: "RESET"
- board text added: "RX"
- board text added: "SCK"
- board text added: "SCL"
- board text added: "SDA"
- board text added: "SS"
- board text added: "TX"

Commit message: Fixed board
Parts:
- removed IMU: IMU, footprints:LGA-14L
- added LSM6DS3US1: IMU, footprints:LGA-14L, F.Cu at (136.3, 111.8)
- MICRO1: footprint footprints:ATMEGA32U4-MUR -> footprints:QFN-44-1EP_7x7mm_Pitch0.5mm_M
Connections:
- U3 pad 12: Net-(U3-Pad12) -> +5V
Routing:
- net /IO11*: track 38.3 -> 23.9 mm
- net /TXLED: track 34.3 -> 27.0 mm
- net GND: track 161.1 -> 154.9 mm
- net /IO9*: track 22.6 -> 28.7 mm, vias 2 -> 3
- net /A3: track 10.7 -> 16.3 mm, vias 0 -> 2
- net +5V: track 110.2 -> 115.6 mm, vias 13 -> 16
- net /SDA_1V8: track 62.6 -> 57.5 mm
- net /IO8: track 56.9 -> 52.1 mm, vias 4 -> 6
- net /A2: track 11.8 -> 16.3 mm, vias 0 -> 2
- net /D4*: track 12.1 -> 16.4 mm, vias 0 -> 2
- net Net-(C2-Pad1): track 5.30 -> 9.59 mm, vias 0 -> 2
- net /A4: track 9.85 -> 14.1 mm, vias 0 -> 2
- net /A1: track 13.5 -> 17.7 mm, vias 0 -> 2
- net /IO10*: track 24.5 -> 28.7 mm
- net Net-(C1-Pad1): track 10.5 -> 14.5 mm
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
Commit message: did DRC
Routing:
- net /TXLED: track 27.0 -> 26.3 mm
