File: CombatBoard/breakout_board2.kicad_pcb (KiCad board)
At the start: 2 copper layers, 50.5 x 30 mm, 36 parts, among them J1 Conn_01x15, J2 Conn_01x15, J3 CONN_02x04, J4 CONN_01X03, J5 Conn_02x03_Odd_Even, J6 Conn_01x02, J7 Conn_01x04, U1 ATMEGA328P-MUR, U2 TB6612FNG, U3 ADP3330, U4 LP5907SNX-3.3/NOPB

Commit message: minot updates
Routing:
- net /D13/SCK: track 64.2 -> 63.3 mm
